File: VNA-Switchboard_FAN3241.kicad_pcb (KiCad board)
At the start: 2 copper layers, 50 x 50 mm, 40 parts, among them J1 6P6C, J2 Conn_01x03_Male, J3 Conn_01x03_Male, J4 Conn_01x02_Male, J5 Conn_01x04_Male, Q1 BC848, Q2 BC807, Q3 BC807, U1 FAN3241, U2 MT3608-PCB

Commit message: R4 and R5 wrong value. C5 larger value optinal.
Parts:
- C5: value 470µ -> 1000µ
- R4: value 22k -> 100k
- R5: value 22k -> 6k2
Other:
- board text added: "Ver. 0.2 2018-12-16"
- board text removed: "Ver. 0.1 2018-11-10"
Changed lines of the file:
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@@
       (effects (font (size 1 1) (thickness 0.15)))
     )
-    (fp_text value 470µ (at 2.5 7.5 270) (layer F.Fab)
+    (fp_text value 1000µ (at 2.5 7.5 270) (layer F.Fab)
       (effects (font (size 1 1) (thickness 0.15)))
     )
@@
       (effects (font (size 1 1) (thickness 0.15)) (justify mirror))
     )
-    (fp_text value 22k (at 0 -1.43 270) (layer B.Fab)
+    (fp_text value 100k (at 0 -1.43 270) (layer B.Fab)
       (effects (font (size 1 1) (thickness 0.15)) (justify mirror))
     )
@@
       (effects (font (size 1 1) (thickness 0.15)) (justify mirror))
     )
-    (fp_text value 22k (at 0 -1.43) (layer B.Fab)
+    (fp_text value 6k2 (at 0 -1.43) (layer B.Fab)
       (effects (font (size 1 1) (thickness 0.15)) (justify mirror))
     )
@@
     (effects (font (size 1.2 1.2) (thickness 0.15)) (justify mirror))
   )
-  (gr_text "Ver. 0.1  2018-11-10" (at 236.601202 91.870248 90) (layer B.SilkS)
+  (gr_text "Ver. 0.2  2018-12-16" (at 236.601202 91.870248 90) (layer B.SilkS)
     (effects (font (size 1.2 1.2) (thickness 0.15)) (justify mirror))
   )
